Commit message: add fork hand model and adjust height

File: robots/hand.xacro (robot description, xacro)
@@ -28,11 +28,15 @@
     <link name="${ns}_leftfinger">
       <visual>
+        <origin xyz="-0.01 -0.01 0" rpy="1.57 3.14 -1.57"/>
         <geometry>
-          <mesh filename="package://franka_panda_description/meshes/visual/finger.dae"/>
+          <mesh filename="/home/asano/Dropbox/CAD/MI-automation/for-robotmodel/panda-hand-tip_heatpress_v2_left.STL" scale="0.001 0.001 0.001"/>
+          <!-- <mesh filename="package://franka_panda_description/meshes/visual/finger.dae"/> -->
         </geometry>
       </visual>
       <collision>
+        <origin xyz="-0.01 -0.01 0" rpy="1.57 3.14 -1.57"/>
         <geometry>
-          <mesh filename="package://franka_panda_description/meshes/collision/finger.stl"/>
+          <mesh filename="/home/asano/Dropbox/CAD/MI-automation/for-robotmodel/panda-hand-tip_heatpress_v2_left.STL" scale="0.001 0.001 0.001"/>
+          <!-- <mesh filename="package://franka_panda_description/meshes/collision/finger.stl"/> -->
         </geometry>
       </collision>
@@ -45,13 +49,15 @@
     <link name="${ns}_rightfinger">
       <visual>
-        <origin xyz="0 0 0" rpy="0 0 ${pi}"/>
+        <origin xyz="-0.01 0.01 0" rpy="-1.57 0 -1.57"/>
         <geometry>
-          <mesh filename="package://franka_panda_description/meshes/visual/finger.dae"/>
+          <mesh filename="/home/asano/Dropbox/CAD/MI-automation/for-robotmodel/panda-hand-tip_heatpress_v2_right.STL" scale="0.001 0.001 0.001"/>
+          <!-- <mesh filename="package://franka_panda_description/meshes/visual/finger.dae"/> -->
         </geometry>
       </visual>
       <collision>
-        <origin xyz="0 0 0" rpy="0 0 ${pi}"/>
+        <origin xyz="0.01 0.01 0" rpy="-1.57 0 -1.57"/>
         <geometry>
-          <mesh filename="package://franka_panda_description/meshes/collision/finger.stl"/>
+          <mesh filename="/home/asano/Dropbox/CAD/MI-automation/for-robotmodel/panda-hand-tip_heatpress_v2_right.STL" scale="0.001 0.001 0.001"/>
+          <!-- <mesh filename="package://franka_panda_description/meshes/collision/finger.stl"/> -->
         </geometry>
       </collision>

File: robots/panda_arm.xacro (robot description, xacro)
@@ -1,5 +1,5 @@
 <?xml version='1.0'?>
 <robot xmlns:xacro="http://www.ros.org/wiki/xacro" name="panda">
-  <xacro:macro name="panda_arm" params="arm_id:='panda' description_pkg:='franka_panda_description' connected_to:='' in_gazebo='false' xyz:='0 0 0' rpy:='0 0 0'">
+  <xacro:macro name="panda_arm" params="arm_id:='panda' description_pkg:='franka_panda_description' connected_to:='' in_gazebo='false' xyz:='0 0 0.6' rpy:='0 0 0'">
     <!-- If using custom frame with ${connected_to} param, make sure 'world' frame exists in its TF tree -->
     <xacro:if value="${connected_to == ''}">
